Commit message: Update floatinghead.urdf

File: urdf/floatinghead.urdf (robot description, URDF)
Before this commit: robot test_model, 3 links, 2 joints
Links:
- added link laser_link
Joints:
- added joint laser_joint: type fixed, parent base_link, child laser_link, origin xyz=0 0.8 0 rpy=0 0 0

Commit message: Update floatinghead.urdf

File: urdf/floatinghead.urdf (robot description, URDF)
Before this commit: robot test_model, 4 links, 3 joints
Links:
- link laser_link: geometry collision sphere radius=.2

Commit message: Update floatinghead.urdf

File: urdf/floatinghead.urdf (robot description, URDF)
Before this commit: robot test_model, 4 links, 3 joints
Joints:
- joint laser_joint: axis (none) -> 0 1 0; origin xyz=0 0.8 0 rpy=0 0 0 -> xyz=0 0 0.8 rpy=0 0 0

Commit message: Update floatinghead.urdf

File: urdf/floatinghead.urdf (robot description, URDF)
Before this commit: robot test_model, 4 links, 3 joints
Links:
- link laser_link: geometry collision sphere radius=.2; visual sphere radius=.2

Commit message: Update floatinghead.urdf

File: urdf/floatinghead.urdf (robot description, URDF)
Before this commit: robot test_model, 4 links, 3 joints
Links:
- link laser_link: geometry collision sphere radius=.2; visual mesh filename=package://floatinghead_description/meshes/pupper.dae

Commit message: Update floatinghead.urdf

File: urdf/floatinghead.urdf (robot description, URDF)
Before this commit: robot test_model, 4 links, 3 joints
Links:
- link base_link: geometry collision cylinder length=0.5 radius=0.25; visual box size=0.2 0.2 1.2

Commit message: Update floatinghead.urdf

File: urdf/floatinghead.urdf (robot description, URDF)
Before this commit: robot test_model, 4 links, 3 joints
Links:
- link laser_link: geometry collision sphere radius=.2; visual mesh filename=package://floatinghead_description/meshes/lidar.dae

Commit message: Update floatinghead.urdf

File: urdf/floatinghead.urdf (robot description, URDF)
Before this commit: robot test_model, 4 links, 3 joints
Links:
- link camera_link: geometry collision mesh filename=package://simpledog/meshes/kinect.dae; visual box size=.1 .1 .1

Commit message: Update floatinghead.urdf

File: urdf/floatinghead.urdf (robot description, URDF)
Before this commit: robot test_model, 4 links, 3 joints
Links:
- link camera_link: geometry collision box size=.1 .1 .1; visual box size=.1 .1 .1

Commit message: Update floatinghead.urdf

File: urdf/floatinghead.urdf (robot description, URDF)
Before this commit: robot test_model, 4 links, 3 joints
Links:
- link base_link: geometry collision cylinder length=0.5 radius=0.25; visual box size=0.2 0.8 .5

Commit message: Update floatinghead.urdf

File: urdf/floatinghead.urdf (robot description, URDF)
Before this commit: robot test_model, 4 links, 3 joints
Joints:
- joint laser_joint: origin xyz=0 0 0.8 rpy=0 0 0 -> xyz=0 0 0.2 rpy=0 0 0

Commit message: Update floatinghead.urdf

File: urdf/floatinghead.urdf (robot description, URDF)
Before this commit: robot test_model, 4 links, 3 joints
Joints:
- joint laser_joint: origin xyz=0 0 0.2 rpy=0 0 0 -> xyz=0 0 -0.2 rpy=0 0 0

Commit message: full lidar range

File: urdf/floatinghead.urdf (robot description, URDF)
Before this commit: robot test_model, 4 links, 3 joints
Joints:
- joint laser_joint: origin xyz=0 0 -0.2 rpy=0 0 0 -> xyz=0 0 0.8 rpy=0 0 0

Commit message: Update floatinghead.urdf

File: urdf/floatinghead.urdf (robot description, URDF)
Before this commit: robot test_model, 5 links, 4 joints
Links:
- added link imu_link; visual sphere radius=0.05
- added link sonic_link_2; visual sphere radius=0.05
- added link sonic_link_3; visual sphere radius=0.05
Joints:
- added joint imu_joint: type fixed, parent base_link, child imu_link, origin xyz=0.0 0.8 0.0 rpy=0 1 0, axis 0 0 0
- added joint sonic_joint_2: type fixed, parent base_link, child sonic_link_2, origin xyz=0.0 0.2 0.0 rpy=0 1 0, axis 0 0 0
- added joint sonic_joint_3: type fixed, parent base_link, child sonic_link_3, origin xyz=0.0 -0.2 0.0 rpy=0 1 0, axis 0 0 0

Commit message: Update floatinghead.urdf

File: urdf/floatinghead.urdf (robot description, URDF)
Before this commit: robot test_model, 8 links, 7 joints
Joints:
- joint imu_joint: origin xyz=0.0 0.8 0.0 rpy=0 1 0 -> xyz=0.0 0.0 0.8 rpy=0 1 0

Commit message: Update floatinghead.urdf

File: urdf/floatinghead.urdf (robot description, URDF)
Before this commit: robot test_model, 8 links, 7 joints
Links:
- added link sonic_link_4; visual sphere radius=0.05
- link base_link: geometry collision box size=2 2 0.75; visual box size=0.9 0.23 .74
Joints:
- added joint sonic_joint_4: type fixed, parent base_link, child sonic_link_4, origin xyz=-0.46 0.0 0.0 rpy=0 2 0, axis 0 0 0
- joint base_link_joint: origin xyz=0.0 0 1.25 rpy=0 0 0 -> xyz=0.0 0 0 rpy=0 0 0

Commit message: Update floatinghead.urdf

File: urdf/floatinghead.urdf (robot description, URDF)
Before this commit: robot test_model, 9 links, 8 joints
Links:
- added link base_link_2, mass 50; collision box size=2 2 0.75; visual box size=0.9 0.23 .74
Joints:
- added joint base_link_joint_rev: type revolute, parent base_link, child base_link_2, origin xyz=0 0 0 rpy=0 0 0, limit lower=-0.0001 upper=0.0001 effort=1000 velocity=1000

Commit message: Update floatinghead.urdf

File: urdf/floatinghead.urdf (robot description, URDF)
Before this commit: robot test_model, 10 links, 9 joints
Links:
- removed link base_link_2
- link base_link: geometry collision box size=0.9 0.23 .74; visual box size=0.9 0.23 .74
Joints:
- removed joint base_link_joint_rev

Commit message: Update floatinghead.urdf

File: urdf/floatinghead.urdf (robot description, URDF)
Before this commit: robot test_model, 9 links, 8 joints
Links:
- link base_link: geometry collision box size=0.9 0.23 .74; visual mesh filename=package://floatinghead_description/meshes/OD.dae
- link sonic_link: geometry visual mesh filename=package://floatinghead_description/meshes/kinect.dae
- link sonic_link_2: geometry visual mesh filename=package://floatinghead_description/meshes/kinect.dae
- link sonic_link_3: geometry visual mesh filename=package://floatinghead_description/meshes/kinect.dae
- link sonic_link_4: geometry visual mesh filename=package://floatinghead_description/meshes/kinect.dae
