Commit message: xacro

File: urdf/floatinghead.urdf.xacro (robot description, xacro)
@@ -1,3 +1,4 @@
-<robot name="test_model">
+<?xml version="1.0"?>
+<robot xmlns:xacro="http://www.ros.org/wiki/xacro">
   <material name="blue1">
     <color rgba="0 0 0.8 1"/>
@@ -393,5 +394,5 @@
     </joint>
     <link name="imu_link">
-    <visual>
+    <!-- <visual>
       <origin xyz="0 0 0" rpy="0 0 0"/>
       <geometry>
@@ -399,5 +400,5 @@
       </geometry>
       <material name="red"/>
-    </visual>
+    </visual> -->
     </link>
     <gazebo reference="imu_link">
@@ -438,5 +439,5 @@
 <!--testing adding the arm urdf-->
   <!-- Include all models -->
-  <xacro:include filename="$(find arm_description)/urdf/Arm_URDF.urdf.xacro"/>
+  <!-- <xacro:include filename="$(find arm_description)/urdf/Arm_URDF.urdf.xacro"/> -->
   <!-- using the models -->
   <!-- <xacro:Arm_URDF base_link="base_link"/>
@@ -444,5 +445,5 @@
   </xacro:Arm_URDF> -->
   <!-- <xacro:include filename = "Arm_URDF.xacro" ns="arm"/> -->
-  <joint name="robot_arm" type="fixed">
+  <!-- <joint name="robot_arm" type="fixed">
     <parent link ="base_link"/>
     <child link = "arm.arm_base_bottom"/>
@@ -450,4 +451,4 @@
     <axis xyz="0  0  0"/>
     <limit effort="1.0" lower="-2.96705973" upper="2.96705973" velocity="1.0"/>
-  </joint>
+  </joint> -->
 </robot>

Commit message: edits

File: urdf/floatinghead.urdf.xacro (robot description, xacro)
@@ -52,12 +52,12 @@
     <minDepth>0.00</minDepth>
   </gazebo>
-  <joint name="camera_joint" type="fixed">
+  <!-- <joint name="camera_joint" type="fixed">
     <axis xyz="0 1 0" />
     <origin xyz="0.25 0.18 0.5" rpy="0 0 0"/>
     <parent link="base_link"/>
     <child link="camera_link"/>
-  </joint>
+  </joint> -->
   <!-- Camera -->
-  <link name="camera_link">
+  <!-- <link name="camera_link">
     <collision>
       <origin xyz="0 0 0" rpy="0 0 0"/>
@@ -78,5 +78,5 @@
       <inertia ixx="1e-6" ixy="0" ixz="0" iyy="1e-6" iyz="0" izz="1e-6" />
     </inertial>
-  </link>
+  </link> -->
   <gazebo>
     <plugin name="object_controller" filename="libgazebo_ros_planar_move.so">
@@ -88,5 +88,5 @@
     </plugin>
   </gazebo>
-   <gazebo reference="camera_link">
+   <!-- <gazebo reference="camera_link">
     <sensor type="camera" name="camera1">
       <update_rate>30.0</update_rate>
@@ -104,7 +104,4 @@
         <noise>
           <type>gaussian</type>
-          <!-- Noise is sampled independently per pixel on each frame.
-               That pixel's noise value is added to each of its color
-               channels, which at that point lie in the range [0,1]. -->
           <mean>0.0</mean>
           <stddev>0.007</stddev>
@@ -126,5 +123,5 @@
       </plugin>
     </sensor>
-  </gazebo>
+  </gazebo> -->
   <joint name="laser_joint" type="fixed">
         <axis xyz="0 0 0" />

File: urdf/floatinghead_overall.urdf (robot description, URDF)
Before this commit: robot floatinghead_model, 14 links, 13 joints
Links:
- removed link camera_link
- added link camera, mass 1; visual box size=0.05 0.05 0.05
Joints:
- removed joint camera_joint
- added joint robot_camera: type fixed, parent base_link, child camera, origin xyz=0.55 0.18 0.38 rpy=0  0  0, axis 0  0  0, limit lower=-2.96705973 upper=2.96705973 effort=1.0 velocity=1.0
- joint robot_arm: origin xyz=0.15 0.18 0.48 rpy=0  0  0 -> xyz=0.35 0.18 0.53 rpy=0  0  0

File: urdf/floatinghead_overall.xacro (robot description, xacro)
@@ -3,8 +3,16 @@
 <xacro:include filename="$(find floatinghead_description)/urdf/floatinghead.urdf.xacro"/>
 <xacro:include filename="$(find arm_description)/urdf/Arm_URDF.xacro"/>
+<xacro:include filename="$(find dcam_description)/urdf/dcam_URDF.xacro"/>
   <joint name="robot_arm" type="fixed">
     <parent link ="base_link"/>
     <child link = "arm_base_bottom"/>
-    <origin rpy="0  0  0" xyz="0.15 0.18 0.48"/>
+    <origin rpy="0  0  0" xyz="0.35 0.18 0.53"/>
+    <axis xyz="0  0  0"/>
+    <limit effort="1.0" lower="-2.96705973" upper="2.96705973" velocity="1.0"/>
+  </joint>
+    <joint name="robot_camera" type="fixed">
+    <parent link ="base_link"/>
+    <child link = "camera"/>
+    <origin rpy="0  0  0" xyz="0.55 0.18 0.38"/>
     <axis xyz="0  0  0"/>
     <limit effort="1.0" lower="-2.96705973" upper="2.96705973" velocity="1.0"/>
